File: pcb/mouse.kicad_pcb (KiCad board)
At the start: 2 copper layers, 70 x 45 mm, 74 parts, among them J1 USB_C_Receptacle_USB2.0, J2 Conn_01x05, J3 Conn_02x03_Counter_Clockwise, J4 Conn_01x06, J5 Conn_01x06, SW1 SW_Push_SPDT, SW2 SW_Push_SPDT, SW3 SW_Push_SPDT, SW4 SW_Push_SPDT, SW5 RotaryEncoder, SW6 SW_Push, U1 pmw3360-t2qu, U2 TLV70018_SOT23-5, U3 STM32F042K6Tx, U4 TLV70033_SOT23-5

Commit message: Updated usb connector placement on pcb
Parts:
- moved J1 1.40 mm to (102.5, 90.0)
Routing:
- net GND: track 420.5 -> 423.3 mm, vias 20 -> 19
- net Net-(J1-PadA6): track 5.36 -> 7.72 mm
- net Net-(J1-PadA7): track 6.30 -> 7.92 mm
- net +5V: track 79.6 -> 80.6 mm, vias 5 -> 4
- net Net-(J1-PadA5): track 7.57 -> 7.05 mm

Commit message: added fabrication files
Other:
- board text added: "github.com/kndndrj"
Changed lines of the file:
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@@
       (layerselection 0x00010fc_ffffffff)
       (disableapertmacros false)
-      (usegerberextensions false)
+      (usegerberextensions true)
       (usegerberattributes true)
-      (usegerberadvancedattributes true)
-      (creategerberjobfile true)
+      (usegerberadvancedattributes false)
+      (creategerberjobfile false)
       (svguseinch false)
       (svgprecision 6)
@@
       (plotinvisibletext false)
       (sketchpadsonfab false)
-      (subtractmaskfromsilk false)
+      (subtractmaskfromsilk true)
       (outputformat 1)
       (mirror false)
-      (drillshape 1)
+      (drillshape 0)
       (scaleselection 1)
-      (outputdirectory "")
+      (outputdirectory "fabrication")
     )
   )
@@
     (property "Sheetname" "buttons")
     (attr smd)
-    (fp_text reference "R8" (at -2.032 -1.524 180) (layer "F.SilkS")
+    (fp_text reference "R8" (at -1.758 -0.198 180) (layer "F.SilkS")
       (effects (font (size 1 1) (thickness 0.15)))
     )
@@
     (property "Sheetname" "buttons")
     (attr smd)
-    (fp_text reference "C15" (at -0.127 -1.27) (layer "F.SilkS")
+    (fp_text reference "C15" (at 0.83 -1.27) (layer "F.SilkS")
       (effects (font (size 1 1) (thickness 0.15)))
     )
@@
     (property "Sheetname" "buttons")
     (attr smd)
-    (fp_text reference "R17" (at 0 -1.27) (layer "F.SilkS")
+    (fp_text reference "R17" (at 1.005 -1.27) (layer "F.SilkS")
       (effects (font (size 1 1) (thickness 0.15)))
     )
@@
     (property "Sheetname" "buttons")
     (attr smd)
-    (fp_text reference "R15" (at 1.524 -1.524 90) (layer "F.SilkS")
+    (fp_text reference "R15" (at -0.147 -1.209 90) (layer "F.SilkS")
       (effects (font (size 1 1) (thickness 0.15)))
     )
@@
   (gr_line (start 167 125) (end 103 125) (layer "Edge.Cuts") (width 0.1))
   (gr_arc (start 103 125) (mid 100.87868 124.12132) (end 100 122) (layer "Edge.Cuts") (width 0.1))
+  (gr_text "github.com/kndndrj" (at 133.5 117.5) (layer "B.SilkS")
+    (effects (font (size 3 3) (thickness 0.5) italic) (justify mirror))
+  )
   (segment (start 105.35 83.49) (end 105.4 83.49) (width 0.6) (layer "F.Cu") (net 1))
   (segment (start 107.244 92.4) (end 106.17 92.4) (width 0.6) (layer "F.Cu") (net 1))
